File: hardware/distance_us.kicad_pcb (KiCad board)
At the start: 2 copper layers, 20 x 45 mm, 26 parts, among them P1 CON-SENSOR, P2 CONN_4, Q1 2N7002P, Q2 2N7002P, U1 LMV358LI, U2 M24C64, U3 DRILL, U4 DRILL, U5 DRILL, U6 DRILL

Commit message: update hardware files
Parts:
- C6: value 0,1µF NC0 -> 0,1µF NP0
Changed lines of the file:
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@@
       (effects (font (size 0.3 0.3) (thickness 0.075)))
     )
-    (fp_text value "0,1µF NC0" (at 0 -0.65 270) (layer F.SilkS)
+    (fp_text value "0,1µF NP0" (at 0 -0.65 270) (layer F.SilkS)
       (effects (font (size 0.3 0.3) (thickness 0.075)))
     )

Commit message: Add 3d information (final)
Parts:
- removed the P2 at (52.9, 42.3)
- added P2: CONN_4, kicad-libraries:pin_array_4x1, F.Cu at (52.9, 42.3)
- added P2: CONN_4, kicad-libraries:distanceUS_overlay, F.Cu at (52.9, 42.3)
- C1, C2, C4, C5, C7, L1: footprint 0603 -> kicad-libraries:C0603
- C3: footprint 0805 -> kicad-libraries:C0805
- C6: footprint 1206 -> kicad-libraries:C1206
- D1: footprint SOD-123 -> kicad-libraries:SOD-123
- P1: footprint CON-SENSOR -> kicad-libraries:CON-SENSOR
- Q1, Q2: footprint SOT23GDS -> kicad-libraries:SOT23GDS
- R1: footprint 0603 -> kicad-libraries:R0603
- RP1: footprint 0603X4 -> kicad-libraries:0603X4
- U1, U2: footprint SOIC8 -> kicad-libraries:SOIC8
- U3, U4, U5, U6: footprint DRILL_NP -> kicad-libraries:DRILL_NP
Connections:
- P1 pad 10: (no net) -> Net-(P1-Pad10)
- RP1 pad 3: (no net) -> Net-(RP1-Pad3)
- RP1 pad 6: (no net) -> Net-(RP1-Pad6)
- U1 pad 1: (no net) -> Net-(U1-Pad1)
- U2 pad 7: (no net) -> Net-(U2-Pad7)
Other:
- outline, holes or cut-outs redrawn
